File: hw/sch_pcb/TTLLVDS01A.kicad_sch (KiCad schematic)
At the start: 17 parts, among them J1 JUMP_3X2, J2 HEADER_2x01_PARALLEL, J3 HEADER_2x01_PARALLEL, J4 HEADER_2x01_PARALLEL, J5 HEADER_2x01_PARALLEL, J6 SATA7-67491-1030, M1 HOLE, M2 HOLE, M3 HOLE, M4 HOLE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

Commit message: Update documentation.
Parts:
- U1: value SN65LVDS9638D -> (none); footprint Package_SO:SOIC-8_3.9x4.9mm_P1.27mm -> (none)
Other:
- note added: "TTL to LVDS (without R3 and R4) SN65LVDS9638D 400 Mbps signalling rate. Operating temperature -40 to 85 SN75LVDS9638D 155 Mbps signalling rate. Operating temperature 0 to 70 LVDS to TTL (with R3 and R4) SN65LVDS9637D SN75LVDS9637D"
- note removed: "TTL to LVDS (without R3 and R4) SN65LVDS9638D SN75LVDS9638D LVDS to TTL (with R3 and R4) SN65LVDS9637D SN75LVDS9637D"
Changed lines of the file:
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@@
   (junction (at 250.19 24.13) (diameter 0) (color 0 0 0 0)
   )
+  (junction (at 242.57 24.13) (diameter 0) (color 0 0 0 0)
+  )
   (junction (at 184.15 91.44) (diameter 0) (color 0 0 0 0)
   )
+  (junction (at 242.57 34.29) (diameter 0) (color 0 0 0 0)
+  )
   (junction (at 171.45 91.44) (diameter 0) (color 0 0 0 0)
   )
@@
     (stroke (width 0) (type default) (color 0 0 0 0))
   )
-  (polyline (pts (xy 237.49 43.18) (xy 237.49 17.78))
+  (polyline (pts (xy 228.6 43.18) (xy 228.6 17.78))
     (stroke (width 0) (type default) (color 0 0 0 0))
   )
@@
     (stroke (width 0) (type default) (color 0 0 0 0))
   )
-  (polyline (pts (xy 278.13 43.18) (xy 237.49 43.18))
+  (polyline (pts (xy 278.13 43.18) (xy 228.6 43.18))
     (stroke (width 0) (type default) (color 0 0 0 0))
   )
@@
     (stroke (width 0) (type default) (color 0 0 0 0))
   )
-  (polyline (pts (xy 237.49 17.78) (xy 278.13 17.78))
+  (polyline (pts (xy 228.6 17.78) (xy 278.13 17.78))
     (stroke (width 0) (type default) (color 0 0 0 0))
   )
@@
     (effects (font (size 1.524 1.524)) (justify left bottom))
   )
-  (text "TTL to LVDS (without R3 and R4)\nSN65LVDS9638D\nSN75LVDS9638D\n\nLVDS to TTL (with R3 and R4)\nSN65LVDS9637D\nSN75LVDS9637D"
+  (text "TTL to LVDS (without R3 and R4)\nSN65LVDS9638D 400 Mbps signalling rate. Operating temperature -40 to 85\nSN75LVDS9638D 155 Mbps signalling rate. Operating temperature 0 to 70\n\nLVDS to TTL (with R3 and R4)\nSN65LVDS9637D\nSN75LVDS9637D"
     (at 170.815 75.565 0)
     (effects (font (size 1.524 1.524)) (justify left bottom))
@@
     (in_bom yes) (on_board yes)
     (property "Reference" "U1" (id 0) (at 147.32 76.2 0))
-    (property "Value" "SN65LVDS9638D" (id 1) (at 153.67 78.74 0))
-    (property "Footprint" "Package_SO:SOIC-8_3.9x4.9mm_P1.27mm" (id 2) (at 144.78 109.22 0)
-      (effects (font (size 1.27 1.27)) hide)
-    )
-    (property "Datasheet" "http://www.ti.com/lit/ds/symlink/ds90lv027a.pdf" (id 3) (at 144.78 82.55 0)
+    (property "Value" "" (id 1) (at 153.67 78.74 0))
+    (property "Footprint" "" (id 2) (at 144.78 109.22 0)
+      (effects (font (size 1.27 1.27)) hide)
+    )
+    (property "Datasheet" "https://www.ti.com/lit/ds/symlink/sn65lvds31.pdf" (id 3) (at 144.78 82.55 0)
       (effects (font (size 1.27 1.27)) hide)
     )
@@
     (pin "2")
   )
+  (symbol (lib_id "power:PWR_FLAG") (at 242.57 24.13 90) (unit 1)
+    (in_bom yes) (on_board yes) (fields_autoplaced)
+    (property "Reference" "#FLG0101" (id 0) (at 240.665 24.13 0)
+      (effects (font (size 1.27 1.27)) hide)
+    )
+    (property "Value" "" (id 1) (at 238.76 24.1299 90)
+      (effects (font (size 1.27 1.27)) (justify left))
+    )
+    (property "Footprint" "" (id 2) (at 242.57 24.13 0)
+      (effects (font (size 1.27 1.27)) hide)
+    )
+    (property "Datasheet" "~" (id 3) (at 242.57 24.13 0)
+      (effects (font (size 1.27 1.27)) hide)
+    )
+    (pin "1")
+  )
+  (symbol (lib_id "power:PWR_FLAG") (at 242.57 34.29 90) (unit 1)
+    (in_bom yes) (on_board yes) (fields_autoplaced)
+    (property "Reference" "#FLG0102" (id 0) (at 240.665 34.29 0)
+      (effects (font (size 1.27 1.27)) hide)
+    )
+    (property "Value" "" (id 1) (at 238.76 34.2899 90)
+      (effects (font (size 1.27 1.27)) (justify left))
+    )
+    (property "Footprint" "" (id 2) (at 242.57 34.29 0)
+      (effects (font (size 1.27 1.27)) hide)
+    )
+    (property "Datasheet" "~" (id 3) (at 242.57 34.29 0)
+      (effects (font (size 1.27 1.27)) hide)
+    )
+    (pin "1")
+  )
   (sheet_instances
     (path "/" (page "1"))
   )
   (symbol_instances
+    (path "/6a13b338-f259-48bd-9888-29f36d488e92"
+      (reference "#FLG0101") (unit 1) (value "PWR_FLAG") (footprint "")
+    )
+    (path "/e271bef5-15e4-40c9-876c-89aee48ff184"
+      (reference "#FLG0102") (unit 1) (value "PWR_FLAG") (footprint "")
+    )
     (path "/00000000-0000-0000-0000-0000549d7353"
       (reference "#PWR01") (unit 1) (value "VCC") (footprint "")

Commit message: Fix title block path issue. Fix submodule versions.
Parts:
- U1: value (none) -> SN65LVDS9638D; footprint (none) -> Package_SO:SOIC-8_3.9x4.9mm_P1.27mm
Changed lines of the file:
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@@
     (in_bom yes) (on_board yes)
     (property "Reference" "U1" (id 0) (at 147.32 76.2 0))
-    (property "Value" "" (id 1) (at 153.67 78.74 0))
-    (property "Footprint" "" (id 2) (at 144.78 109.22 0)
+    (property "Value" "SN65LVDS9638D" (id 1) (at 153.67 78.74 0))
+    (property "Footprint" "Package_SO:SOIC-8_3.9x4.9mm_P1.27mm" (id 2) (at 144.78 109.22 0)
       (effects (font (size 1.27 1.27)) hide)
     )
@@
       (effects (font (size 1.27 1.27)) hide)
     )
-    (property "Value" "" (id 1) (at 238.76 24.1299 90)
+    (property "Value" "PWR_FLAG" (id 1) (at 238.76 24.1299 90)
       (effects (font (size 1.27 1.27)) (justify left))
     )
@@
       (effects (font (size 1.27 1.27)) hide)
     )
-    (property "Value" "" (id 1) (at 238.76 34.2899 90)
-      (effects (font (size 1.27 1.27)) (justify left))
-    )
+    (property "Value" "PWR_FLAG" (id 1) (at 238.76 34.2899 90)
+      (effects (font (size 1.27 1.27)) (justify left))
+    )

Commit message: Zmena pouzder na nova KiCAD a poslední kontroly pred vyrobou
Parts:
- C2, R1, R2, R3, R4: footprint Mlab_R:SMD-0805 -> Resistor_SMD:R_0805_2012Metric
Changed lines of the file:
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@@
       (effects (font (size 1.27 1.27)) (justify left))
     )
-    (property "Footprint" "Mlab_R:SMD-0805" (id 2) (at 250.19 29.21 0)
+    (property "Footprint" "Resistor_SMD:R_0805_2012Metric" (id 2) (at 250.19 29.21 0)
       (effects (font (size 1.524 1.524)) hide)
     )
@@
       (effects (font (size 1.27 1.27)) (justify left))
     )
-    (property "Footprint" "Mlab_R:SMD-0805" (id 2) (at 169.672 87.63 90)
+    (property "Footprint" "Resistor_SMD:R_0805_2012Metric" (id 2) (at 169.672 87.63 90)
       (effects (font (size 1.27 1.27)) hide)
     )
@@
       (effects (font (size 1.27 1.27)) (justify left))
     )
-    (property "Footprint" "Mlab_R:SMD-0805" (id 2) (at 169.672 97.79 90)
+    (property "Footprint" "Resistor_SMD:R_0805_2012Metric" (id 2) (at 169.672 97.79 90)
       (effects (font (size 1.27 1.27)) hide)
     )
@@
       (effects (font (size 1.27 1.27)) (justify left))
     )
-    (property "Footprint" "Mlab_R:SMD-0805" (id 2) (at 113.03 85.852 90)
+    (property "Footprint" "Resistor_SMD:R_0805_2012Metric" (id 2) (at 113.03 85.852 90)
       (effects (font (size 1.27 1.27)) hide)
     )
@@
       (effects (font (size 1.27 1.27)) (justify left))
     )
-    (property "Footprint" "Mlab_R:SMD-0805" (id 2) (at 113.03 96.012 90)
+    (property "Footprint" "Resistor_SMD:R_0805_2012Metric" (id 2) (at 113.03 96.012 90)
       (effects (font (size 1.27 1.27)) hide)
     )
@@
     )
     (path "/00000000-0000-0000-0000-00005562302c"
-      (reference "C2") (unit 1) (value "100nF") (footprint "Mlab_R:SMD-0805")
+      (reference "C2") (unit 1) (value "100nF") (footprint "Resistor_SMD:R_0805_2012Metric")
     )
     (path "/00000000-0000-0000-0000-00005b4de0b5"
@@
     )
     (path "/00000000-0000-0000-0000-00005c6cc9e7"
-      (reference "R1") (unit 1) (value "33R") (footprint "Mlab_R:SMD-0805")
+      (reference "R1") (unit 1) (value "33R") (footprint "Resistor_SMD:R_0805_2012Metric")
     )
     (path "/00000000-0000-0000-0000-00005c6ccb45"
-      (reference "R2") (unit 1) (value "33R") (footprint "Mlab_R:SMD-0805")
+      (reference "R2") (unit 1) (value "33R") (footprint "Resistor_SMD:R_0805_2012Metric")
     )
     (path "/00000000-0000-0000-0000-00005c6beb35"
-      (reference "R3") (unit 1) (value "100") (footprint "Mlab_R:SMD-0805")
+      (reference "R3") (unit 1) (value "100") (footprint "Resistor_SMD:R_0805_2012Metric")
     )
     (path "/00000000-0000-0000-0000-00005c6becc5"
-      (reference "R4") (unit 1) (value "100") (footprint "Mlab_R:SMD-0805")
+      (reference "R4") (unit 1) (value "100") (footprint "Resistor_SMD:R_0805_2012Metric")
     )
     (path "/00000000-0000-0000-0000-00005c6be27c"

Commit message: Priprava podkladu pro vyrobu
Parts:
- C2: value 100nF -> (none); footprint Resistor_SMD:R_0805_2012Metric -> (none); UST_ID (none) -> 5c70984712875079b91f8b4c
- D1: value BZV55C-3,6V -> (none); footprint Diode_SMD:D_MiniMELF -> (none); UST_ID (none) -> 5c70984512875079b91f88b1
- J1: value JUMP_3X2 -> (none); footprint Mlab_Pin_Headers:Straight_2x03 -> (none)
- J2, J3, J4, J5: value HEADER_2x01_PARALLEL -> (none); footprint Mlab_Pin_Headers:Straight_2x01 -> (none)
- J6: value SATA7-67491-1030 -> (none); footprint Mlab_CON:SATA-7_THT_VERT_2 -> (none)
- M1, M2, M3, M4: value HOLE -> (none); footprint Mlab_Mechanical:MountingHole_3mm -> (none)
- R1, R2: value 33R -> (none); footprint Resistor_SMD:R_0805_2012Metric -> (none)
- R3, R4: value 100 -> (none); footprint Resistor_SMD:R_0805_2012Metric -> (none)
- U1: value SN65LVDS9638D -> (none); footprint Package_SO:SOIC-8_3.9x4.9mm_P1.27mm -> (none)
Changed lines of the file:
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@@
       (effects (font (size 1.524 1.524)))
     )
-    (property "Value" "HOLE" (id 1) (at 257.81 48.26 0)
-      (effects (font (size 1.524 1.524)) hide)
-    )
-    (property "Footprint" "Mlab_Mechanical:MountingHole_3mm" (id 2) (at 255.27 48.26 0)
+    (property "Value" "" (id 1) (at 257.81 48.26 0)
+      (effects (font (size 1.524 1.524)) hide)
+    )
+    (property "Footprint" "" (id 2) (at 255.27 48.26 0)
       (effects (font (size 1.524 1.524)) hide)
     )
@@
       (effects (font (size 1.524 1.524)))
     )
-    (property "Value" "HOLE" (id 1) (at 262.89 48.26 0)
-      (effects (font (size 1.524 1.524)) hide)
-    )
-    (property "Footprint" "Mlab_Mechanical:MountingHole_3mm" (id 2) (at 260.35 48.26 0)
+    (property "Value" "" (id 1) (at 262.89 48.26 0)
+      (effects (font (size 1.524 1.524)) hide)
+    )
+    (property "Footprint" "" (id 2) (at 260.35 48.26 0)
       (effects (font (size 1.524 1.524)) hide)
     )
@@
       (effects (font (size 1.524 1.524)))
     )
-    (property "Value" "HOLE" (id 1) (at 267.97 48.26 0)
-      (effects (font (size 1.524 1.524)) hide)
-    )
-    (property "Footprint" "Mlab_Mechanical:MountingHole_3mm" (id 2) (at 265.43 48.26 0)
+    (property "Value" "" (id 1) (at 267.97 48.26 0)
+      (effects (font (size 1.524 1.524)) hide)
+    )
+    (property "Footprint" "" (id 2) (at 265.43 48.26 0)
       (effects (font (size 1.524 1.524)) hide)
     )
@@
       (effects (font (size 1.524 1.524)))
     )
-    (property "Value" "HOLE" (id 1) (at 273.05 48.26 0)
-      (effects (font (size 1.524 1.524)) hide)
-    )
-    (property "Footprint" "Mlab_Mechanical:MountingHole_3mm" (id 2) (at 270.51 48.26 0)
+    (property "Value" "" (id 1) (at 273.05 48.26 0)
+      (effects (font (size 1.524 1.524)) hide)
+    )
+    (property "Footprint" "" (id 2) (at 270.51 48.26 0)
       (effects (font (size 1.524 1.524)) hide)
     )
@@
       (effects (font (size 1.27 1.27)) (justify left))
     )
-    (property "Value" "100nF" (id 1) (at 250.19 31.75 0)
-      (effects (font (size 1.27 1.27)) (justify left))
-    )
-    (property "Footprint" "Resistor_SMD:R_0805_2012Metric" (id 2) (at 250.19 29.21 0)
+    (property "Value" "" (id 1) (at 250.19 31.75 0)
+      (effects (font (size 1.27 1.27)) (justify left))
+    )
+    (property "Footprint" "" (id 2) (at 250.19 29.21 0)
       (effects (font (size 1.524 1.524)) hide)
     )
@@
       (effects (font (size 1.27 1.27)) hide)
     )
+    (property "UST_ID" "5c70984712875079b91f8b4c" (id 5) (at 250.19 29.21 0)
+      (effects (font (size 1.27 1.27)) hide)
+    )
     (pin "1")
     (pin "2")
@@
       (effects (font (size 1.27 1.27)) (justify left))
     )
-    (property "Value" "JUMP_3X2" (id 1) (at 276.86 24.13 90)
+    (property "Value" "" (id 1) (at 276.86 24.13 90)
       (effects (font (size 1.016 1.016)) hide)
     )
-    (property "Footprint" "Mlab_Pin_Headers:Straight_2x03" (id 2) (at 276.86 25.4 0)
+    (property "Footprint" "" (id 2) (at 276.86 25.4 0)
       (effects (font (size 1.524 1.524)) hide)
     )
@@
       (effects (font (size 1.27 1.27)) (justify left))
     )
-    (property "Value" "BZV55C-3,6V" (id 1) (at 257.81 31.75 90)
-      (effects (font (size 1.27 1.27)) (justify left))
-    )
-    (property "Footprint" "Diode_SMD:D_MiniMELF" (id 2) (at 257.81 29.21 0)
+    (property "Value" "" (id 1) (at 257.81 31.75 90)
+      (effects (font (size 1.27 1.27)) (justify left))
+    )
+    (property "Footprint" "" (id 2) (at 257.81 29.21 0)
       (effects (font (size 1.524 1.524)) hide)
     )
@@
       (effects (font (size 1.524 1.524)))
     )
+    (property "UST_ID" "5c70984512875079b91f88b1" (id 4) (at 257.81 29.21 0)
+      (effects (font (size 1.27 1.27)) hide)
+    )
     (pin "1")
     (pin "2")
@@
     (in_bom yes) (on_board yes)
     (property "Reference" "U1" (id 0) (at 147.32 76.2 0))
-    (property "Value" "SN65LVDS9638D" (id 1) (at 153.67 78.74 0))
-    (property "Footprint" "Package_SO:SOIC-8_3.9x4.9mm_P1.27mm" (id 2) (at 144.78 109.22 0)
+    (property "Value" "" (id 1) (at 153.67 78.74 0))
+    (property "Footprint" "" (id 2) (at 144.78 109.22 0)
       (effects (font (size 1.27 1.27)) hide)
     )
@@
       (effects (font (size 1.27 1.27)) (justify left))
     )
-    (property "Value" "SATA7-67491-1030" (id 1) (at 195.0212 92.583 0)
-      (effects (font (size 1.27 1.27)) (justify left))
-    )
-    (property "Footprint" "Mlab_CON:SATA-7_THT_VERT_2" (id 2) (at 191.77 87.63 0)
+    (property "Value" "" (id 1) (at 195.0212 92.583 0)
+      (effects (font (size 1.27 1.27)) (justify left))
+    )
+    (property "Footprint" "" (id 2) (at 191.77 87.63 0)
       (effects (font (size 1.27 1.27)) hide)
     )
@@
       (effects (font (size 1.27 1.27)) (justify left))
     )
-    (property "Value" "100" (id 1) (at 171.45 89.535 90)
-      (effects (font (size 1.27 1.27)) (justify left))
-    )
-    (property "Footprint" "Resistor_SMD:R_0805_2012Metric" (id 2) (at 169.672 87.63 90)
+    (property "Value" "" (id 1) (at 171.45 89.535 90)
+      (effects (font (size 1.27 1.27)) (justify left))
+    )
+    (property "Footprint" "" (id 2) (at 169.672 87.63 90)
       (effects (font (size 1.27 1.27)) hide)
     )
@@
       (effects (font (size 1.27 1.27)) (justify left))
     )
-    (property "Value" "100" (id 1) (at 171.45 99.695 90)
-      (effects (font (size 1.27 1.27)) (justify left))
-    )
-    (property "Footprint" "Resistor_SMD:R_0805_2012Metric" (id 2) (at 169.672 97.79 90)
+    (property "Value" "" (id 1) (at 171.45 99.695 90)
+      (effects (font (size 1.27 1.27)) (justify left))
+    )
+    (property "Footprint" "" (id 2) (at 169.672 97.79 90)
       (effects (font (size 1.27 1.27)) hide)
     )
@@
       (effects (font (size 1.524 1.524)))
     )
-    (property "Value" "HEADER_2x01_PARALLEL" (id 1) (at 93.4974 84.3026 0)
-      (effects (font (size 1.524 1.524)) hide)
-    )
-    (property "Footprint" "Mlab_Pin_Headers:Straight_2x01" (id 2) (at 91.44 87.63 0)
+    (property "Value" "" (id 1) (at 93.4974 84.3026 0)
+      (effects (font (size 1.524 1.524)) hide)
+    )
+    (property "Footprint" "" (id 2) (at 91.44 87.63 0)
       (effects (font (size 1.524 1.524)) hide)
     )
@@
       (effects (font (size 1.524 1.524)))
     )
-    (property "Value" "HEADER_2x01_PARALLEL" (id 1) (at 93.4974 86.8426 0)
-      (effects (font (size 1.524 1.524)) hide)
-    )
-    (property "Footprint" "Mlab_Pin_Headers:Straight_2x01" (id 2) (at 91.44 90.17 0)
+    (property "Value" "" (id 1) (at 93.4974 86.8426 0)
+      (effects (font (size 1.524 1.524)) hide)
+    )
+    (property "Footprint" "" (id 2) (at 91.44 90.17 0)
       (effects (font (size 1.524 1.524)) hide)
     )
@@
       (effects (font (size 1.524 1.524)))
     )
-    (property "Value" "HEADER_2x01_PARALLEL" (id 1) (at 93.4974 94.4626 0)
-      (effects (font (size 1.524 1.524)) hide)
-    )
-    (property "Footprint" "Mlab_Pin_Headers:Straight_2x01" (id 2) (at 91.44 97.79 0)
+    (property "Value" "" (id 1) (at 93.4974 94.4626 0)
+      (effects (font (size 1.524 1.524)) hide)
+    )
+    (property "Footprint" "" (id 2) (at 91.44 97.79 0)
       (effects (font (size 1.524 1.524)) hide)
     )
@@
       (effects (font (size 1.524 1.524)))
     )
-    (property "Value" "HEADER_2x01_PARALLEL" (id 1) (at 93.4974 97.0026 0)
-      (effects (font (size 1.524 1.524)) hide)
-    )
-    (property "Footprint" "Mlab_Pin_Headers:Straight_2x01" (id 2) (at 91.44 100.33 0)
+    (property "Value" "" (id 1) (at 93.4974 97.0026 0)
+      (effects (font (size 1.524 1.524)) hide)
+    )
+    (property "Footprint" "" (id 2) (at 91.44 100.33 0)
       (effects (font (size 1.524 1.524)) hide)
     )
@@
       (effects (font (size 1.27 1.27)) (justify left))
     )
-    (property "Value" "33R" (id 1) (at 110.49 87.63 90)
-      (effects (font (size 1.27 1.27)) (justify left))
-    )
-    (property "Footprint" "Resistor_SMD:R_0805_2012Metric" (id 2) (at 113.03 85.852 90)
+    (property "Value" "" (id 1) (at 110.49 87.63 90)
+      (effects (font (size 1.27 1.27)) (justify left))
+    )
+    (property "Footprint" "" (id 2) (at 113.03 85.852 90)
       (effects (font (size 1.27 1.27)) hide)
     )
@@
       (effects (font (size 1.27 1.27)) (justify left))
     )
-    (property "Value" "33R" (id 1) (at 110.49 97.79 90)
-      (effects (font (size 1.27 1.27)) (justify left))
-    )
-    (property "Footprint" "Resistor_SMD:R_0805_2012Metric" (id 2) (at 113.03 96.012 90)
-      (effects (font (size 1.27 1.27)) hide)
-    )
+    (property "Value" "" (id 1) (at 110.49 97.79 90)
+      (effects (font (size 1.27 1.27)) (justify left))
+    )
+    (property "Footprint" "" (id 2) (at 113.03 96.012 90)
+      (effects (font (size 1.27 1.27)) hide)
+    )
